Commit message: fixing bench collsion mesh

File: models/stage.urdf.xacro (robot description, xacro)
@@ -6,7 +6,7 @@
     <origin xyz="0 0 0" rpy="0 0 0" />
     <parent link="world"/>
-    <child link="bench_link"/>
+    <child link="stage_link"/>
   </joint>
-  <link name = "bench_link">
+  <link name = "stage_link">
     <inertial>
       <origin xyz="0 0 0" />
