Commit message: adding shadow generator, fixing shadowless mesh

File: models/manipulation_platform.urdf.xacro (robot description, xacro)
@@ -19,5 +19,5 @@
         <origin rpy="0 0 0 " xyz="0 0 0"/>
         <geometry>
-          <mesh filename="package://lcsr_barrett/models/meshes/manipulation_platform.dae"/>
+          <mesh filename="package://lcsr_barrett/models/meshes/manipulation_platform.stl"/>
         </geometry>
       </visual>

Commit message: added color to platform

File: models/manipulation_platform.urdf.xacro (robot description, xacro)
@@ -21,4 +21,7 @@
           <mesh filename="package://lcsr_barrett/models/meshes/manipulation_platform.stl"/>
         </geometry>
+        <material name="white">
+          <color rgba="0.75 0.80 1 1"/>
+        </material>
       </visual>
       <collision>

Commit message: reducing d-gains for pid with hand, adding some colors to the environment

File: models/manipulation_platform.urdf.xacro (robot description, xacro)
@@ -18,4 +18,5 @@
       <visual>
         <origin rpy="0 0 0 " xyz="0 0 0"/>
+        <material>Gazebo/DarkGrey</material>
         <geometry>
           <mesh filename="package://lcsr_barrett/models/meshes/manipulation_platform.stl"/>

Commit message: adding platform material

File: models/manipulation_platform.urdf.xacro (robot description, xacro)
@@ -2,34 +2,41 @@
   xmlns:xacro="http://www.ros.org/wiki/xacro">
   <link name="world"/>
-    <joint name="platform_link_fixed_joint"  type="fixed">
-      <origin xyz="0 0 0" rpy="0 0 0" />
-      <parent link="world"/>
-      <child link="platform_link"/>
-    </joint>
-    <link name = "platform_link">
-      <inertial>
-        <origin xyz="0 0 0" />
-        <mass value="25" />
-        <inertia
-          ixx="1" ixy="0"   ixz="0"
-                  iyy="1"   iyz="0"
-                            izz="1" />
-      </inertial>
-      <visual>
-        <origin rpy="0 0 0 " xyz="0 0 0"/>
-        <geometry>
-          <mesh filename="package://lcsr_barrett/models/meshes/manipulation_platform.stl"/>
-        </geometry>
-      </visual>
-      <collision>
-        <origin rpy="0 0 0 " xyz="0 0 0"/>
-        <geometry>
-          <mesh filename="package://lcsr_barrett/models/meshes/manipulation_platform.stl"/>
-        </geometry>
-      </collision>
-    </link>
-    <gazebo reference="platform_link">
-      <kp>50000</kp>
-      <kd>8</kd>
-    </gazebo>
+  <joint name="platform_link_fixed_joint"  type="fixed">
+    <origin xyz="0 0 0" rpy="0 0 0" />
+    <parent link="world"/>
+    <child link="platform_link"/>
+  </joint>
+  <link name = "platform_link">
+    <inertial>
+      <origin xyz="0 0 0" />
+      <mass value="25" />
+      <inertia
+        ixx="1" ixy="0"   ixz="0"
+        iyy="1"   iyz="0"
+        izz="1" />
+    </inertial>
+    <visual>
+      <origin rpy="0 0 0 " xyz="0 0 0"/>
+      <geometry>
+        <mesh filename="package://lcsr_barrett/models/meshes/manipulation_platform.stl"/>
+      </geometry>
+    </visual>
+    <collision>
+      <origin rpy="0 0 0 " xyz="0 0 0"/>
+      <geometry>
+        <mesh filename="package://lcsr_barrett/models/meshes/manipulation_platform.stl"/>
+      </geometry>
+    </collision>
+  </link>
+  <gazebo reference="platform_link">
+    <kp>50000</kp>
+    <kd>8</kd>
+    <visual name="visual">
+      <material>
+        <ambient>0 0 0 0</ambient>
+        <specular>0.8 0.8 0.8 0.1</specular>
+        <diffuse>1.0 1.0 1.0 1.0</diffuse>
+      </material>
+    </visual>
+  </gazebo>
 </robot>

Commit message: added manipulation platform color

File: models/manipulation_platform.urdf.xacro (robot description, xacro)
@@ -18,4 +18,7 @@
     <visual>
       <origin rpy="0 0 0 " xyz="0 0 0"/>
+      <material name="white">
+        <color rgba="0.8 0.8 0.8 1"/>
+      </material>
       <geometry>
         <mesh filename="package://lcsr_barrett/models/meshes/manipulation_platform.stl"/>
