Commit message: numerous outstanding changes

File: launch/sim/wam7_sim.urdf.xacro (robot description, xacro)
@@ -12,5 +12,5 @@
     </plugin>
     <plugin name="gazebo_ros_moveit_planning_scene" filename="libgazebo_ros_moveit_planning_scene.so">
-      <robotNamespace>~</robotNamespace>
+      <robotNamespace>/gazebo</robotNamespace>
       <sceneName>B08</sceneName>
       <robotName>wam</robotName>

File: models/manipulation_platform.urdf.xacro (robot description, xacro)
@@ -19,5 +19,5 @@
         <origin rpy="0 0 0 " xyz="0 0 0"/>
         <geometry>
-          <mesh filename="package://lcsr_barrett/models/meshes/manipulation_platform.stl"/>
+          <mesh filename="package://lcsr_barrett/models/meshes/platform.stl"/>
         </geometry>
       </visual>
@@ -25,5 +25,5 @@
         <origin rpy="0 0 0 " xyz="0 0 0"/>
         <geometry>
-          <mesh filename="package://lcsr_barrett/models/meshes/manipulation_platform.stl"/>
+          <mesh filename="package://lcsr_barrett/models/meshes/platform.stl"/>
         </geometry>
       </collision>
